File: schematic/pi-pico-vga.kicad_sch (KiCad schematic)
At the start: 33 parts, among them J1 VGA, J2 USB Keyboard, J3 Micro_SD_Card, J4 Power, J5 UART, J6 External, J8 AudioJack4, SW1 Power switch, SW2 User, SW3 Microswitch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

Commit message: .
Parts:
- removed C1: 0.1uF, symbol Device:C
- removed C2: 10uF, symbol Device:C_Polarized
- removed J8: AudioJack4, symbol Connector_Audio:AudioJack4
- removed R9: 1k, symbol Device:R
- added J7: Passive Buzzer, symbol Connector_Generic:Conn_01x03
Connections:
- net +5V: now also J7.1 (Pin_1)
- net AUDIO: now also RV2.1
- net GND: now also J7.3 (Pin_3); no longer RV2.3
- net at RV2.2: now also J7.2 (Pin_2)
- no-connect marks 23 -> 24
Other:
- moved on the sheet: J2, RV2
